File: led-matrix/LEDMatrixLearningBadge.brd (EAGLE design)
At the start: 100.3 x 48.8 mm, 96 parts, among them IC1 5M40ZE64, IC2 MEGA48/88/168-MU, Q1 HM4522P-423-G, SW1 4_DIRECTIONAL_JOYSTICK_PLUS_C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, T1 ZXM61P03, T10 ZXM61P03, T11 ZXM61P03, T12 ZXM61P03, T13 ZXM61P03, T14 ZXM61P03, T15 ZXM61P03, T16 ZXM61P03, T17 DMN65D8L, T18 DMN65D8L, T19 DMN65D8L, T2 ZXM61P03, T20 DMN65D8L, T21 DMN65D8L, T22 DMN65D8L, T23 DMN65D8L, T24 DMN65D8L, T25 DMN65D8L, T26 DMN65D8L, T27 DMN65D8L, T28 DMN65D8L, T29 DMN65D8L, T3 ZXM61P03, T30 DMN65D8L, T31 DMN65D8L, T32 DMN65D8L, T4 ZXM61P03, T5 ZXM61P03, T6 ZXM61P03, T7 ZXM61P03, T8 ZXM61P03, T9 ZXM61P03, U1 FT440-FIXED, U2 MCP6L01, Y1 8MHz

Commit message: Signal rename
Renamed CPLD signals to cpu to reflect reworked hdl code
Connections:
- net COLUMN0 renamed ROW_ENABLE_FROM_CPU
- net COLUMN1 renamed GREEN_ROW_FROM_CPU_DATA
- net COLUMN2 renamed RED_ROW_FROM_CPU_DATA
- net COLUMN3 renamed ROW_FROM_CPU_CLK
- net ROW_CLK renamed COLUMN_CLK
- net ROW_DATA renamed COLUMN_DATA
Changed lines of the file:
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@@
 <wire x1="19.9384" y1="23.5712" x2="19.9136" y2="23.5712" width="0.2032" layer="1"/>
 </signal>
-<signal name="ROW_DATA">
+<signal name="COLUMN_DATA">
 <contactref element="IC1" pad="38"/>
 <contactref element="IC2" pad="10"/>
@@
 <wire x1="32.45" y1="15.0988" x2="33.528" y2="14.0208" width="0.2032" layer="16"/>
 </signal>
-<signal name="ROW_CLK">
+<signal name="COLUMN_CLK">
 <contactref element="IC1" pad="40"/>
 <contactref element="IC2" pad="9"/>
@@
 <wire x1="32.95" y1="16.0212" x2="34.544" y2="14.4272" width="0.2032" layer="16"/>
 </signal>
-<signal name="COLUMN0">
+<signal name="ROW_ENABLE_FROM_CPU">
 <contactref element="IC2" pad="11"/>
 <via x="32.512" y="13.6144" extent="1-16" drill="0.4064" diameter="0.4064"/>
@@
 <wire x1="31.95" y1="14.1764" x2="32.512" y2="13.6144" width="0.2032" layer="16"/>
 </signal>
-<signal name="COLUMN1">
+<signal name="GREEN_ROW_FROM_CPU_DATA">
 <contactref element="IC2" pad="12"/>
 <via x="31.496" y="13.208" extent="1-16" drill="0.4064" diameter="0.4064"/>
@@
 <wire x1="31.45" y1="13.254" x2="31.496" y2="13.208" width="0.2032" layer="16"/>
 </signal>
-<signal name="COLUMN2">
+<signal name="RED_ROW_FROM_CPU_DATA">
 <contactref element="IC2" pad="13"/>
 <via x="30.48" y="12.8016" extent="1-16" drill="0.4064" diameter="0.4064"/>
@@
 <wire x1="30.48" y1="13.4112" x2="30.48" y2="12.8016" width="0.2032" layer="16"/>
 </signal>
-<signal name="COLUMN3">
+<signal name="ROW_FROM_CPU_CLK">
 <contactref element="IC2" pad="14"/>
 <via x="29.464" y="12.3952" extent="1-16" drill="0.4064" diameter="0.4064"/>
