File: ethernet-gateway/ethernetGateway.sch (EAGLE design)
At the start: 56 parts, among them IC1 IC_ENC28J60-SOIC-28, IC2 REG1117, IC3 IC_FT230X-SSOP-16, J1 MAGJACK, J3 AVR_SPI_PRG_6PTH, U2 ATMEGA328P

Commit message: Update ethernet gateway reset circuit
Parts:
- removed R16: 10k, rcl:R-EU_R0805
- R7: value 2k32 -> 6k8
Connections:
- net 3V3: no longer R16.1
- net N$20: no longer R16.2
Changed lines of the file:
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@@
 <part name="SUPPLY8" library="supply2" deviceset="GND" device=""/>
 <part name="JP2" library="pinhead" deviceset="PINHD-2X10" device=""/>
-<part name="R7" library="rcl" deviceset="R-EU_" device="R0805" value="2k32"/>
+<part name="R7" library="rcl" deviceset="R-EU_" device="R0805" value="6k8"/>
 <part name="J3" library="SparkFun-Connectors" deviceset="AVR_SPI_PRG_6" device="PTH"/>
 <part name="R9" library="rcl" deviceset="R-EU_" device="R0805" value="2k32"/>
@@
 <part name="R15" library="rcl" deviceset="R-EU_" device="R0805" value="10k"/>
 <part name="C18" library="rcl" deviceset="C-EU" device="C0805" value="0.1uF"/>
-<part name="R16" library="rcl" deviceset="R-EU_" device="R0805" value="10k"/>
 </parts>
 <sheets>
@@
 <instance part="R15" gate="G$1" x="142.24" y="-25.4" rot="R270"/>
 <instance part="C18" gate="G$1" x="139.7" y="-43.18" rot="R270"/>
-<instance part="R16" gate="G$1" x="127" y="-25.4" rot="R270"/>
 </instances>
 <busses>
@@
 <label x="137.16" y="-15.24" size="1.778" layer="95"/>
 <junction x="134.62" y="-20.32"/>
-<pinref part="R16" gate="G$1" pin="1"/>
-<wire x1="127" y1="-20.32" x2="134.62" y2="-20.32" width="0.1524" layer="91"/>
 </segment>
 </net>
@@
 <pinref part="C18" gate="G$1" pin="2"/>
 <wire x1="134.62" y1="-38.1" x2="134.62" y2="-43.18" width="0.1524" layer="91"/>
-<pinref part="R16" gate="G$1" pin="2"/>
-<wire x1="127" y1="-30.48" x2="127" y2="-38.1" width="0.1524" layer="91"/>
 <pinref part="IC3" gate="IC" pin="!RTS"/>
-<wire x1="127" y1="-38.1" x2="134.62" y2="-38.1" width="0.1524" layer="91"/>
-<wire x1="124.46" y1="-38.1" x2="127" y2="-38.1" width="0.1524" layer="91"/>
-<junction x="127" y="-38.1"/>
-</segment>
-</net>
+<wire x1="124.46" y1="-38.1" x2="134.62" y2="-38.1" width="0.1524" layer="91"/>
+</segment>
+</net>
