File: maker-faire-2013/circle.brd (EAGLE design)
At the start: 45.7 x 45.7 mm, 14 parts, among them Q1 2N3904, Q2 2N3904, SW1 0S102011MS2QN1

Commit message: 2015 MF PCB final
Connections:
- removed net CASE1: BATTERY.1, SW1.1, SW1.2, SW1.CASE1
- new net 1: SW1.1
- new net N$1: BATTERY.1, SW1.2
- net CASE2: now also SW1.CASE1
Routing:
- net CASE1: track 34.2 -> 0.00 mm, vias 1 -> 0
- net N$1: track 0.00 -> 32.4 mm, vias 0 -> 1
Other:
- board text added: "v2.2"
- board text removed: "v2.0"
Changed lines of the file:
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@@
 <setting verticaltext="up"/>
 </settings>
-<grid distance="0.0125" unitdist="inch" unit="inch" style="dots" multiple="1" display="yes" altdistance="0.05" altunitdist="inch" altunit="inch"/>
+<grid distance="0.00625" unitdist="inch" unit="inch" style="dots" multiple="1" display="yes" altdistance="0.05" altunitdist="inch" altunit="inch"/>
 <layers>
 <layer number="1" name="Top" color="4" fill="1" visible="yes" active="yes"/>
@@
 <circle x="21.59" y="20.955" radius="22.86" width="0.4064" layer="20"/>
 <text x="20.955" y="5.08" size="2.794" layer="25" font="vector" ratio="10" rot="SR180" align="center">hackspace.ca</text>
-<text x="20.955" y="0.3175" size="2.794" layer="26" font="vector" ratio="10" rot="SMR180" align="center">v2.0</text>
+<text x="20.955" y="0.3175" size="2.794" layer="26" font="vector" ratio="10" rot="SMR180" align="center">v2.2</text>
 </plain>
 <attributes>
@@
 </class>
 </classes>
-<designrules name="dirt_cheap_dirty_boards.v1">
-<description language="en">&lt;b&gt;Dirty Cheap Dirty Board Design Rules&lt;/b&gt;
-&lt;br&gt;
-&lt;br&gt;Min width/Spacing: 5/5mil
-&lt;br&gt;Min diameter of finished hole 12mil</description>
+<designrules name="iteadstudio_drc">
+<description language="de">&lt;b&gt;EAGLE Design Rules&lt;/b&gt;
+&lt;p&gt;
+Die Standard-Design-Rules sind so gewählt, dass sie für
+die meisten Anwendungen passen. Sollte ihre Platine
+besondere Anforderungen haben, treffen Sie die erforderlichen
+Einstellungen hier und speichern die Design Rules unter
+einem neuen Namen ab.</description>
+<description language="en">&lt;b&gt;EAGLE Design Rules&lt;/b&gt;
+&lt;p&gt;
+The default Design Rules have been set to cover
+a wide range of applications. Your particular design
+may have different requirements, so please make the
+necessary adjustments and save your customized
+design rules under a new name.</description>
+<description language="zh">&lt;b&gt;Seeed Studio EAGLE Design Rules&lt;/b&gt;
+</description>
 <param name="layerSetup" value="(1*16)"/>
-<param name="mtCopper" value="0.035mm 0.0175mm 0.035mm 0.035mm 0.035mm 0.035mm 0.035mm 0.035mm 0.035mm 0.035mm 0.035mm 0.035mm 0.035mm 0.035mm 0.0175mm 0.035mm"/>
-<param name="mtIsolate" value="1.5mm 1.1mm 0.2mm 0.15mm 0.2mm 0.15mm 0.2mm 0.15mm 0.2mm 0.15mm 0.2mm 0.15mm 0.2mm 0.15mm 0.2mm"/>
-<param name="mdWireWire" value="5mil"/>
-<param name="mdWirePad" value="5mil"/>
-<param name="mdWireVia" value="5mil"/>
-<param name="mdPadPad" value="5mil"/>
-<param name="mdPadVia" value="5mil"/>
-<param name="mdViaVia" value="5mil"/>
+<param name="mtCopper" value="0.035mm 0.035mm 0.035mm 0.035mm 0.035mm 0.035mm 0.035mm 0.035mm 0.035mm 0.035mm 0.035mm 0.035mm 0.035mm 0.035mm 0.035mm 0.035mm"/>
+<param name="mtIsolate" value="1.5mm 0.15mm 0.2mm 0.15mm 0.2mm 0.15mm 0.2mm 0.15mm 0.2mm 0.15mm 0.2mm 0.15mm 0.2mm 0.15mm 0.2mm"/>
+<param name="mdWireWire" value="6mil"/>
+<param name="mdWirePad" value="6mil"/>
+<param name="mdWireVia" value="6mil"/>
+<param name="mdPadPad" value="6mil"/>
+<param name="mdPadVia" value="6mil"/>
+<param name="mdViaVia" value="6mil"/>
 <param name="mdSmdPad" value="0mil"/>
 <param name="mdSmdVia" value="0mil"/>
@@
 <param name="mdDrill" value="10mil"/>
 <param name="mdSmdStop" value="0mil"/>
-<param name="msWidth" value="5mil"/>
+<param name="msWidth" value="6mil"/>
 <param name="msDrill" value="12mil"/>
 <param name="msMicroVia" value="12mil"/>
@@
 <param name="mlMinCreamFrame" value="0mil"/>
 <param name="mlMaxCreamFrame" value="0mil"/>
-<param name="mlViaStopLimit" value="25mil"/>
+<param name="mlViaStopLimit" value="100mil"/>
 <param name="srRoundness" value="0"/>
 <param name="srMinRoundness" value="0mil"/>
@@
 <via x="1.5875" y="29.5275" extent="1-16" drill="0.6" shape="octagon"/>
 <via x="10.795" y="29.5275" extent="1-16" drill="0.6" shape="octagon"/>
-</signal>
-<signal name="CASE1">
-<contactref element="SW1" pad="2"/>
-<contactref element="BATTERY" pad="1"/>
-<contactref element="SW1" pad="1"/>
-<contactref element="SW1" pad="CASE1"/>
-<wire x1="21.59" y1="36.51" x2="24.1275" y2="33.9725" width="1.27" layer="1"/>
-<wire x1="24.1275" y1="33.9725" x2="24.13" y2="33.9725" width="1.27" layer="1"/>
-<wire x1="26.035" y1="10.795" x2="25.781" y2="10.795" width="1.27" layer="1"/>
-<wire x1="25.781" y1="10.795" x2="23.681" y2="10.795" width="1.27" layer="1"/>
-<wire x1="21.681" y1="10.795" x2="23.681" y2="10.795" width="1.27" layer="1"/>
-<wire x1="24.1275" y1="33.9725" x2="24.1275" y2="32.3875" width="1.27" layer="1"/>
-<wire x1="24.1275" y1="32.3875" x2="28.575" y2="27.94" width="1.27" layer="1"/>
-<via x="28.575" y="27.94" extent="1-16" drill="0.6" shape="octagon"/>
-<wire x1="28.575" y1="27.94" x2="28.575" y2="26.3525" width="1.27" layer="16"/>
-<wire x1="28.575" y1="26.3525" x2="26.035" y2="23.8125" width="1.27" layer="16"/>
-<wire x1="25.7175" y1="10.8585" x2="25.781" y2="10.795" width="1.27" layer="16"/>
-<wire x1="26.035" y1="23.8125" x2="26.035" y2="11.049" width="1.27" layer="16"/>
-<wire x1="26.035" y1="11.049" x2="25.781" y2="10.795" width="1.27" layer="16"/>
+<via x="24.765" y="28.8925" extent="1-16" drill="0.6" shape="octagon"/>
 </signal>
 <signal name="CASE2">
@@
 <wire x1="33.581278125" y1="33.692646875" x2="31.077353125" y2="33.692646875" width="1.27" layer="1"/>
 <wire x1="31.077353125" y1="33.692646875" x2="29.21" y2="35.56" width="1.27" layer="1"/>
+<contactref element="SW1" pad="CASE1"/>
+</signal>
+<signal name="N$1">
+<contactref element="SW1" pad="2"/>
+<contactref element="BATTERY" pad="1"/>
+<wire x1="21.681" y1="10.795" x2="21.681" y2="11.521" width="1.016" layer="16"/>
+<wire x1="21.681" y1="11.521" x2="23.01875" y2="12.85875" width="0.762" layer="16"/>
+<wire x1="23.01875" y1="12.85875" x2="23.495" y2="12.85875" width="0.762" layer="16"/>
+<wire x1="23.495" y1="12.85875" x2="25.4" y2="14.76375" width="0.762" layer="16"/>
+<wire x1="25.4" y1="14.76375" x2="25.87625" y2="15.24" width="1.016" layer="16"/>
+<wire x1="25.87625" y1="15.24" x2="25.87625" y2="23.65375" width="1.016" layer="16"/>
+<wire x1="25.87625" y1="23.65375" x2="28.73375" y2="26.51125" width="1.016" layer="16"/>
+<wire x1="28.73375" y1="26.51125" x2="28.73375" y2="28.09875" width="1.016" layer="16"/>
+<via x="28.73375" y="28.09875" extent="1-16" drill="0.6" shape="octagon"/>
+<wire x1="28.73375" y1="28.09875" x2="27.78125" y2="28.09875" width="1.016" layer="1"/>
+<wire x1="27.78125" y1="28.09875" x2="21.59" y2="34.29" width="1.016" layer="1"/>
+<wire x1="21.59" y1="34.29" x2="21.59" y2="36.51" width="1.016" layer="1"/>
+</signal>
+<signal name="1">
+<contactref element="SW1" pad="1"/>
 </signal>
 </signals>
