File: arduino-leonardo-eagle-workshop/Arduino_Leonardo-REV3b/Arduino_Leonardo-REV3b.sch (EAGLE design)
At the start: 51 parts, among them IC1 NCP1117ST50T3G, IC2 LMV358IDGKR, J1 USB MICRO, J2 8x1F-H8.5, J3 8x1F-H8.5, J4 6x1F-H8.5, T1 FDN340P, U1 ATMEGA32U4-XUMU, U2 ATMEGA32U4-XUAU, U3 LP2985-33DBVR, Y1 16MHz KX-7

Commit message: Updates
Parts:
- removed C10, C12: 10u, rcl:CPOL-EUSMCB
- removed C11, C14: 1u, SmartPrj:C-EUC0603
- removed C22: 100n, SmartPrj:C-EUC0603
- removed D1: M7, diode:DIODE-SMB
- removed EXTPOWER: POWERSUPPLY_DC21MMX, SmartPrj:POWERSUPPLY_DC21MMX
- removed IC1: NCP1117ST50T3G, linear:MC33269ST-3.3T3
- removed IC2: LMV358IDGKR, linear:LMV358MMX
- removed J1: USB MICRO, SmartPrj:MYCON2_USB-MINI-B
- removed J3: 8x1F-H8.5, SmartPrj:PINHD-1X8
- removed J4: 6x1F-H8.5, SmartPrj:PINHD-1X6
- removed JP1: 10x1F-H8.5, SmartPrj:PINHD-1X10
- removed ORIGIN: TP_SP, SmartPrj:TP_SP
- removed RN2: 1K, resistor-dil:4R-NCAY16
- removed RN3: 22R, resistor-dil:4R-NCAY16
- removed T1: FDN340P, zetex:PMOSSOT23
- removed U1: ATMEGA32U4-XUMU, SmartPrj:ATMEGA32U4-XUMU
- removed U3: LP2985-33DBVR, SmartPrj:LP2985-XXDBVR33
- removed Z1, Z2: CG0603MLC-05E, varistor:VARISTORCN0603
- added R4, R5, R6, R7: 1k, rcl:R-EU_R0805
- added R8, R9: 22R, rcl:R-EU_R0805
- J2: value 8x1F-H8.5 -> USB-MINIB-5PIN; device SmartPrj:PINHD-1X8 -> SparkFun-Connectors:USB-MINIB-5PIN
Connections:
- removed net +3V3: C14.2, IC2B.-IN, J3.4, U3.OUT
- removed net CMP: C22.2, IC2B.+IN, RN1A.2, RN1B.2
- removed net GATE_CMD: IC2B.OUT, T1.G
- removed net LL: IC2A.-IN, IC2A.OUT, RN2B.1
- removed net N$6: RN2C.2, TX.A
- removed net N$8: RN2D.2, RX.A
- removed net VIN: C10.+, D1.C, EXTPOWER.2, IC1.IN, J3.8, RN1A.1
- new net N$1: L.A, R4.1
- new net N$4: R6.1, RX.A
- net +5V: now also R4.2, R5.2, R6.2, R7.2; no longer C11.2, C12.+, IC1.OUT, IC1.OUT@1, IC2P.V+, J3.2, J3.5, RN2A.1, RN2C.1, RN2D.1, T1.S, U1.UVCC, U1.VCC, U1.VCC1, U3.IN, U3.ON/!OFF
- net A0: no longer J4.1, U1.(ADC7/TDI)PF7
- net A1: no longer J4.2, U1.(ADC6/TDO)PF6
- net A2: no longer J4.3, U1.(ADC5/TMS)PF5
- net A3: no longer J4.4, U1.(ADC4/TCK)PF4
- net A4: no longer J4.5, U1.(ADC1)PF1
- net A5: no longer J4.6, U1.(ADC0)PF0
- net AGND: no longer U1.GND3
- net AREF: no longer JP1.8, U1.AREF
- net AVCC: no longer U1.AVCC, U1.AVCC1
- net D+: now also J2.D+, R9.1; no longer J1.D+, RN3A.2, Z1.1
- net D-: now also J2.D-, R8.1; no longer J1.D-, RN3D.2, Z2.1
- net D0/RX: no longer J2.1, U1.(RXD1/AIN1/INT2)PD2
- net D1/TX: no longer J2.2, U1.(TXD1/INT3)PD3
- net D2/SDA: no longer J2.3, JP1.9, U1.(SDA/INT1)PD1
- net D3/SCL: no longer J2.4, JP1.10, U1.(OC0B/SCL/INT0)PD0
- net D4: no longer J2.5, U1.(ICP1/ADC8)PD4
- net D5*: no longer J2.6, U1.(OC3A/#0C4A)PC6
- net D6*: no longer J2.7, U1.(T0/OC4D/ADC10)PD7
- net D7: no longer J2.8, U1.(INT6/AIN0)PE6
- net GND: now also J2.MTN1, J2.MTN2, J2.MTN3, J2.MTN4; no longer C10.-, C11.1, C12.-, C14.1, C22.1, D1.A, EXTPOWER.1, EXTPOWER.3, IC1.GND/ADJ, IC2P.V-, J1.SH1, J1.SH2, J1.SH3, J1.SH4, J1.SH5, J1.SH6, J3.6, J3.7, JP1.7, L.C, RN1B.1, U1.GND, U1.GND1, U1.GND2, U1.PAD, U3.GND, Z1.2, Z2.2
- net HWB: no longer U1.(#HWB)PE2
- net IO10*: no longer JP1.3, U1.(PCINT6/OC1B/OC4B/ADC13)PB6
- net IO11*: no longer JP1.4, U1.(PCINT7/OC0A/OC1C/#RTS)PB7
- net IO12: no longer JP1.5, U1.(T1/#OC4D/ADC9)PD6
- net IO13*: now also L.C; no longer IC2A.+IN, JP1.6, U1.(ICP3/CLK0/OC4A)PC7
- net IO8: no longer JP1.1, U1.(ADC11/PCINT4)PB4
- net IO9*: no longer JP1.2, U1.(PCINT5/OC1A/#OC4B/ADC12)PB5
- net MISO: no longer U1.(PD0/MISO/PCINT3)PB3
- net MOSI: no longer U1.(PDI/MOSI/PCINT2)PB2
- net N$2: now also R5.1, TX.A; no longer L.A, RN2B.2
- net N$3: now also R7.1; no longer RN2A.2
- net RD+: now also R9.2; no longer RN3A.1, U1.D+
- net RD-: now also R8.2; no longer RN3D.1, U1.D-
- net RESET: no longer J3.3, U1.RESET
- net RXLED: no longer U1.(SS/PCINT0)PB0
- net SCK: no longer U1.(SCLK/PCINT1)PB1
- net TXLED: no longer U1.(XCK1/#CTS)PD5
- net UCAP: no longer U1.UCAP
- net UGND: now also J2.GND; no longer J1.GND, U1.UGND
- net USBID: now also J2.ID; no longer J1.ID
- net VUSB: no longer T1.D, U1.VBUS
- net XTAL1: no longer U1.XTAL1
- net XTAL2: no longer U1.XTAL2
- net XUSB: now also J2.VBUS; no longer J1.VBUS
Other:
- note removed: "+5V AUTO SELECTOR"
- note removed: "10"
- note removed: "11"
- note removed: "3"
- note removed: "5"
- note removed: "6"
- note removed: "9"
- note removed: "Arduino LEONARDO"
- note removed: "IOREF"
- note removed: "NOT USED"
- note removed: "RFU"
- note removed: "TM"
- moved on the sheet: C13, L, L2, ON, RN1C, RX, TX, U2

Commit message: Add copies of sparkfun and adafruit libraries Add FET and PWM output to schematic
Parts:
- removed FID1, FID2, FID3: FIDUCIALMOUNT, SmartPrj:FIDUCIALMOUNT
- added JP2: SERVO-OUT, SparkFun-Connectors:M031X03_NO_SILK
- added Q1: FDMA1024NZ, PEBBLE:FDMA1024NZ
- added R10: 1k, SparkFun:RESISTOR0402-RES
- added SL1: (no value), con-amp-quick:M02
Connections:
- new net N$17: Q1A.D, Q1A.D1, SL1.2
- net +5V: now also JP2.2, SL1.1
- net D6*: now also JP2.3
- net D7: now also Q1A.G, R10.2
- net GND: now also JP2.1, Q1A.S, R10.1
Other:
- note added: "Servo Motor Output"
